File: static/AquaLux.kicad_sch (KiCad schematic)
At the start: 0 parts

Commit message: fixed a variety of issues, including wifi credential storage, logging, threshold setting, light detection, etc.
Parts:
- added B2: ~, symbol Custom_symbols:B5109
- added BT1: Battery, symbol Device:Battery
- added BZ1: Buzzer, symbol Device:Buzzer
- added Q1: NPN, symbol Simulation_SPICE:NPN
- added R1: R_Photo, symbol Device:R_Photo
- added R2: R, symbol Device:R
- added U1: ESP32-S2, Package_DFN_QFN:QFN-56-1EP_7x7mm_P0.4mm_EP4x4mm, symbol MCU_Espressif:ESP32-S2
Connections:
- new net: R1.1, R2.2, U1.28 (GPIO21)
- new net: B2. (IN-), BT1.1 (+)
- new net: B2. (IN-), BT1.2 (-)
- new net: U1.1 (VDDA), U1.51 (VDDA), U1.54 (VDDA)
- new net: U1.3 (VDD3P3), U1.4 (VDD3P3)
- new net: Q1.2 (B), U1.42 (GPIO38)
- new net: BZ1.2 (-), Q1.3 (E)
- new net +3V8: R2.1

Commit message: added kicad schematics properly.
Parts:
- removed B2: ~, symbol Custom_symbols:B5109
- removed R1: R_Photo, symbol Device:R_Photo
- removed R2: R, symbol Device:R
- added B1: ~, symbol Custom_symbols:B5109
- added BT2: Battery, symbol Device:Battery
- added Capacitance_Pad1: ~, symbol Custom_symbols:Capacitance_Pad
- added Photoresistor1: ~, symbol Custom_symbols:Photoresistor
- added TP1: ~, symbol Custom_symbols:TP4056
Connections:
- net at U1.28 (GPIO21): now also Photoresistor1. (GND)
- net at BT1.1 (+): now also TP1. (IN-)
- net at BT1.2 (-): now also TP1. (IN-)
- net at U1.10 (GPIO5): now also Capacitance_Pad1.
- net at U1.3 (VDD3P3), U1.4 (VDD3P3): now also B1. (IN-)
- net at U1.57 (GND): now also Q1.1 (C), B1. (IN-), Photoresistor1. (GND), TP1. (IN-)
- net at BZ1.1 (+): now also Photoresistor1. (GND), TP1. (IN-)
- new net: B1. (IN-), BT2.1 (+)
- new net: B1. (IN-), BT2.2 (-)
Other:
- company: (none) -> Adyansh
- title: (none) -> Aqualux circuit diagram
- moved on the sheet: BT1, BZ1, Q1, U1
