File: static/AquaLux.kicad_sch (KiCad schematic)
At the start: 9 parts, among them Q1 NPN, U1 ESP32-S2

Commit message: Normalise line endings
Connections:
- new net: B1. (IN-), Photoresistor1. (GND), Q1.1 (C), TP1. (IN-), U1.57 (GND)
- now unconnected: B1. (IN-), TP1. (IN-)
